File: iso_analog/iso_analog.kicad_pcb (KiCad board)
At the start: 2 copper layers, 64 x 33 mm, 29 parts, among them J1 Conn_01x02_Socket, J2 Conn_01x02_Socket, J3 Conn_01x02_Socket, J4 Conn_01x02_Socket, U2 LM321, U3 LM321

Commit message: iso analog update stuff
Parts:
- removed D1: 5.1V, Diode_SMD:D_SOD-323_HandSoldering
- removed R4: 1k, RMC_Resistor:R_0805_2012Metric_Pad1.20x1.40mm_HandSolder_L
- added C5: 0.1uF, RMC_Capacitor:C_0805_2012Metric_Pad1.18x1.45mm_HandSolder_L, F.Cu at (136.6, 75.5)
- added C6: 0.1uF, RMC_Capacitor:C_0805_2012Metric_Pad1.18x1.45mm_HandSolder_L, F.Cu at (159.1, 72.5)
- added D2: LED, RMC_LED:LED_0805_2012Metric_Pad1.45x1.40mm_HandSolder, F.Cu at (166.1, 58.6)
- added D3: LED, RMC_LED:LED_0805_2012Metric_Pad1.45x1.40mm_HandSolder, F.Cu at (139.4, 58.4)
- added R5: 1k, RMC_Resistor:R_0805_2012Metric_Pad1.20x1.40mm_HandSolder_L, F.Cu at (166.1, 56.1)
- added R6: 1k, RMC_Resistor:R_0805_2012Metric_Pad1.20x1.40mm_HandSolder_L, F.Cu at (139.4, 56.1)
- JP1: footprint Connector_PinHeader_2.54mm:PinHeader_1x03_P2.54mm_Vertical -> Jumper:SolderJumper-3_P1.3mm_Open_Pad1.0x1.5mm
- JP2: footprint Connector_PinHeader_2.54mm:PinHeader_1x02_P2.54mm_Vertical -> Jumper:SolderJumper-2_P1.3mm_Open_Pad1.0x1.5mm
- R1: value 1k -> 100
- R2, R3: value 10k -> 100k
- moved JP1 2.51 mm to (124.5, 74.9), turned to -90 degrees
- moved R2 2.40 mm to (136.6, 78.9)
- moved JP2 2.39 mm to (128.2, 59.3), turned to 0 degrees
- moved R3 1.00 mm to (159.1, 76.0), turned to 180 degrees
Connections:
- JP1 pad 1: Net-(D1-K) -> Net-(J1-Pin_1)
- R2 pad 2: Net-(U1-C1) -> Net-(U1-A1)
- R3 pad 2: Net-(U1-C2) -> Net-(U1-A2)
- RV1 pad 1: +5V -> GND
- RV1 pad 3: GND -> +5V
- TP3 pad 1: Net-(U1-C1) -> Net-(U1-A1)
- TP4 pad 1: Net-(U1-C2) -> Net-(U1-A2)
- U1 pad 3: Net-(U1-C1) -> +5V
- U1 pad 4: +5V -> Net-(U1-A1)
- U1 pad 5: +5VA -> Net-(U1-A2)
- U1 pad 6: Net-(U1-C2) -> +5VA
- U2 pad 3: Net-(U1-C1) -> Net-(U1-A1)
- U3 pad 1: Net-(U1-C2) -> Net-(U1-A2)
Routing:
- net Net-(U1-A1): track 0.00 -> 39.4 mm, vias 0 -> 2
- net Net-(U1-C1): track 31.0 -> 0.00 mm, vias 2 -> 0
- net Net-(U1-A2): track 0.00 -> 23.5 mm
- net Net-(U1-C2): track 22.6 -> 0.00 mm
- net Net-(J1-Pin_1): track 5.19 -> 14.7 mm
- net Net-(D1-K): track 8.59 -> 0.00 mm
- net +5V: track 96.1 -> 87.8 mm, vias 1 -> 2
- net Net-(JP1-C): track 25.4 -> 17.5 mm
- net +5VA: track 66.1 -> 62.0 mm, vias 2 -> 0
- net Net-(D2-K): track 0.00 -> 2.41 mm
- net Net-(D3-K): track 0.00 -> 2.34 mm
- net Net-(JP2-B): track 18.6 -> 16.8 mm
- net Net-(JP1-B): track 8.89 -> 9.42 mm
- net GND: vias 0 -> 1
Other:
- outline, holes or cut-outs redrawn
- board text added: "ISO Analog Dev v1.1 2026/01/19"
- board text removed: "ISO Analog Dev v1.0 2026/01/13"
