File: iso_analog/iso_analog.kicad_sch (KiCad schematic)
At the start: 29 parts, among them J1 Conn_01x02_Socket, J2 Conn_01x02_Socket, J3 Conn_01x02_Socket, J4 Conn_01x02_Socket, U2 LM321, U3 LM321

Commit message: iso analog update stuff
Parts:
- removed D1: 5.1V, Diode_SMD:D_SOD-323_HandSoldering, symbol Device:D_Zener
- removed R4: 1k, RMC_Resistor:R_0805_2012Metric_Pad1.20x1.40mm_HandSolder_L, symbol Device:R
- added C5, C6: 0.1uF, RMC_Capacitor:C_0805_2012Metric_Pad1.18x1.45mm_HandSolder_L, symbol Device:C
- added D2, D3: LED, RMC_LED:LED_0805_2012Metric_Pad1.45x1.40mm_HandSolder, symbol Device:LED
- added R5, R6: 1k, RMC_Resistor:R_0805_2012Metric_Pad1.20x1.40mm_HandSolder_L, symbol Device:R
- JP1: footprint Connector_PinHeader_2.54mm:PinHeader_1x03_P2.54mm_Vertical -> Jumper:SolderJumper-3_P1.3mm_Open_Pad1.0x1.5mm
- JP2: footprint Connector_PinHeader_2.54mm:PinHeader_1x02_P2.54mm_Vertical -> Jumper:SolderJumper-2_P1.3mm_Open_Pad1.0x1.5mm
- R1: value 1k -> 100
- R2, R3: value 10k -> 100k
Connections:
- net +5V: now also RV1.3, U1.3 (C1), D3.2 (A); no longer RV1.1, U1.4 (A1)
- net +5VA: now also U1.6 (C2), D2.2 (A); no longer U1.5 (A2)
- net GND: now also RV1.1, C5.2, R6.1; no longer RV1.3
- net GND1: now also C6.2, R5.1
- net at R2.2, TP3.1, U2.3 (-): now also U1.4 (A1), C5.1; no longer U1.3 (C1)
- net at R3.2, TP4.1, U3.1 (+): now also U1.5 (A2), C6.1; no longer U1.6 (C2)
- net at JP1.1 (A): now also J1.1 (Pin_1)
- new net: D2.1 (K), R5.2
- new net: D3.1 (K), R6.2
Other:
- moved on the sheet: TP4
